File: 2.3/DCP23.brd (EAGLE design)
At the start: 0 parts

Commit message: blah
Parts:
- added C1, C2: 18pF, C_digikey:C0603
- added CON1: USB-1, Connectors:MICRO_USB_WITH_PEGS
- added IC1: STM32F103CBT7, stm32:LQFP48
- added IC2: AP2127-3.3, linear regulators:SOT23-5
- added LED0, LED1, LED2, LED3: LED-0603, rc:LED0603
- added Q1: 8 MHz, crystal:OSCILLATOR-5.0X3.2-4P
- added R1, R2, R3, R4: 1K, R_digikey:R0603
Connections:
- new net GND: C1.P$2, C2.P$2, IC2.2, LED0.C, LED1.C, LED2.C, LED3.C, Q1.2, Q1.4
- new net LED0: IC1.20, R3.P$2
- new net LED1: IC1.21, R1.P$2
- new net LED2: IC1.22, R2.P$2
- new net N$1: C1.P$1, IC1.5, Q1.1
- new net N$2: LED0.A, R3.P$1
- new net N$3: C2.P$1, IC1.6, Q1.3
- new net N$4: LED2.A, R2.P$1
- new net N$5: LED1.A, R1.P$1
- new net N$6: LED3.A, R4.P$1
- new net SWITCH: IC1.25
- new net VBUS: IC1.26
- new net VDD_3V3: IC2.5, R4.P$2
- new net VDD_5V: IC2.1, IC2.3
Other:
- board outline added: 40 x 20 mm

Commit message: 2.3 schematic  completed
Parts:
- added C10, C11, C12, C13, C14, C17, C18, C19, C6, C7, C8, C9: 0.1µF, C_digikey:C0603
- added C15: 1µF, C_digikey:C0603
- added C16: 10nF, C_digikey:C0603
- added C3, C4, C5: 4.7µF, C_digikey:C0603
- added CON2: PINHEAD_1X02-2, pinhead:1X02-PTH-2
- added CON3: CON-6P-SM06B, Connectors:SM06B
- added CON4: CON-2X5P, Connectors:200215-00010T1LF
- added CON5: CON-6P-DF13, Connectors:DF13C-6P-1.25V
- added CON6: PINHEAD_1X04-2.54, pinhead:1X04-PTH-2.54
- added CON7: PINHEAD_1X03-2.54, pinhead:1X03-PTH-2.54
- added CON8: PINHEAD_1X06-2.54, pinhead:1X06-PTH-2.54
- added D1: PRTR5V0U2X, TVS_diodes:SOT143B
- added IC3, IC4, IC5, IC6: 74LVC2T45, misc:VSSOP8
- added Q2: DMG1023UV-7, mosfet:SOT-563
- added Q3: DMG1024UV-7, mosfet:SOT-563
- added R10: 4K7, R_digikey:R0603
- added R11, R12, R13, R14, R24: 10K, R_digikey:R0603
- added R15, R16, R17, R18, R19, R20, R21, R23: 120R, R_digikey:R0603
- added R22: 0, R_digikey:R0603
- added R5, R6: 22R, rc:R0603
- added R7: 1K5, rc:R0603
- added SW1: TACT_SWITCH-FSMSM, misc:FSMSM
- moved IC2 51.0 mm to (-25.0, 30.0)
- moved LED0 51.0 mm to (-25.0, 10.0)
- moved LED1 51.0 mm to (-25.0, 25.0)
- moved LED2 51.0 mm to (-25.0, 20.0)
- moved LED3 51.0 mm to (-25.0, 0.00)
- moved R1 51.0 mm to (-25.0, 35.0)
- moved R2 51.0 mm to (-25.0, 15.0)
- moved R3 51.0 mm to (-25.0, 5.00)
- moved R4 51.0 mm to (-25.0, -5.00)
Connections:
- removed net VBUS: IC1.26
- new net !RST: IC1.7
- new net CONSOLE_RX: CON3.3, CON5.5, CON8.3, R23.P$2
- new net CONSOLE_TX: CON3.2, CON5.4, CON8.2, R20.P$2
- new net IRST: IC1.12, Q3.5
- new net IRST_SENSE: IC1.17, Q3.6
- new net IRXD: IC1.31, IC5.3
- new net ITCK: IC1.15, IC4.2
- new net ITDI: IC1.13, IC4.3
- new net ITDO: IC1.16, IC5.2
- new net ITMS: IC1.14, IC6.3
- new net ITMS_DIR: IC1.11, IC6.5
- new net ITXD: IC1.30, IC3.3
- new net N$10: CON1.D-, CON6.2, R6.2
- new net N$11: CON1.D+, CON6.1, R5.2
- new net N$12: Q2.1, Q2.4, R14.P$1
- new net N$13: CON5.1, R22.P$2
- new net N$15: CON2.1, IC1.44, R12.P$1
- new net N$7: IC1.29, R7.1
- new net N$8: D1.3, IC1.32, R6.1
- new net N$9: D1.2, IC1.33, R5.1, R7.2
- new net PWR_BR: IC1.19, Q2.2, Q2.5, R14.P$2
- new net RST: CON4.10, R15.P$2
- new net SWCLK: CON7.3, IC1.37
- new net SWDIO: CON7.1, IC1.34
- new net TCK: CON3.5, CON4.4, CON8.5, R18.P$2
- new net TDI: CON4.8, R16.P$2
- new net TDO: CON4.6, R17.P$2
- new net TMS: CON3.4, CON4.2, CON8.4, R19.P$2
- new net TPWR: CON3.1, CON4.1, CON8.1, Q2.6, R10.P$2, R21.P$2
- new net TRACESWO: IC1.39
- new net VBUS1: C6.P$2, IC1.18, R10.P$1, R11.P$2
- new net XRST: Q3.2, Q3.3, R13.P$1, R15.P$1
- new net XRXD: IC5.6, R20.P$1
- new net XTCK: IC4.7, R18.P$1
- new net XTDI: IC4.6, R16.P$1
- new net XTDO: IC5.7, R17.P$1
- new net XTMS: IC6.6, R19.P$1
- new net XTPWR: C11.P$2, C12.P$2, C13.P$2, C14.P$2, IC3.8, IC4.8, IC5.8, IC6.8, R13.P$2, R21.P$1
- new net XTXD: IC3.6, R23.P$1
- net GND: now also C10.P$2, C11.P$1, C12.P$1, C13.P$1, C14.P$1, C15.P$1, C16.P$1, C17.P$2, C18.P$1, C19.P$2, C3.P$1, C4.P$1, C5.P$2, C6.P$1, C7.P$2, C8.P$2, C9.P$2, CON1.GND, CON3.6, CON3.G1, CON3.G2, CON4.3, CON4.5, CON4.9, CON5.G1, CON5.G2, CON6.4, CON7.2, CON8.6, D1.1, IC1.23, IC1.35, IC1.8, IC3.2, IC3.4, IC3.7, IC4.4, IC5.4, IC5.5, IC6.2, IC6.4, IC6.7, Q3.1, Q3.4, R11.P$1, R12.P$2, SW1.P$2
- net SWITCH: now also R24.P$1, SW1.P$1
- net VDD_3V3: now also C10.P$1, C15.P$2, C16.P$2, C17.P$1, C18.P$2, C19.P$1, C4.P$2, C5.P$1, C7.P$1, C8.P$1, C9.P$1, CON2.2, IC1.1, IC1.24, IC1.36, IC1.40, IC1.41, IC1.42, IC1.48, IC1.9, IC3.1, IC3.5, IC4.1, IC4.5, IC5.1, IC6.1, Q2.3, R24.P$2
- net VDD_5V: now also C3.P$2, CON1.VBUS, CON6.3, D1.4, IC1.26, R22.P$1

Commit message: Some routing
Parts:
- added D2: BAT30SWFILM, Diodes:SC70
- moved R24 137.6 mm to (2.75, -5.25)
- moved CON7 132.2 mm to (11.0, 8.50), turned to 180 degrees
- moved SW1 125.8 mm to (7.50, -7.25)
- moved CON8 124.5 mm to (-28.5, -1.25), turned to 90 degrees
- moved R23 117.9 mm to (-15.0, 2.50)
- moved R22 113.8 mm to (-11.8, 3.00)
- moved R21 112.7 mm to (-19.0, 12.5)
- moved CON6 110.7 mm to (15.0, 0.00), turned to 270 degrees
- moved CON5 102.3 mm to (-15.5, 7.25), turned to 180 degrees
- moved CON4 82.0 mm to (-18.8, -3.00), turned to 270 degrees
- moved R19 75.9 mm to (-13.2, 0.00), turned to 180 degrees
- moved R20 70.3 mm to (-12.8, -10.8), turned to 180 degrees
- moved R18 69.5 mm to (-13.2, -1.50), turned to 180 degrees
- moved CON3 63.6 mm to (-36.2, 11.5), turned to 270 degrees
- moved R13 63.3 mm to (-11.5, 13.0), turned to 90 degrees
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Connections:
- net GND: now also CON6.1, D2.1; no longer CON6.4
- net N$10: now also CON6.3; no longer CON6.2
- net N$11: now also CON6.2; no longer CON6.1
- net VBUS1: now also D2.3
- net VDD_3V3: now also D2.2
- net VDD_5V: now also CON6.4; no longer CON6.3
Other:
- board size 40 x 20 mm -> 45 x 20 mm
- board text added: "DCP2.2 dimensions 44x22"

Commit message: more routing
Parts:
- removed CON8: PINHEAD_1X06-2.54, pinhead:1X06-PTH-2.54
- added CON10: PINHEAD_2X03-PTH-2.54, pinhead:2X03-PTH-2.54
- moved R20 20.9 mm to (-5.78, 9.00)
- moved Q2 17.5 mm to (-23.7, 16.8)
- moved R14 17.5 mm to (-21.4, 16.7)
- moved CON3 15.6 mm to (-26.2, -0.50)
- moved C11 11.1 mm to (-15.8, -12.2)
- moved C6 10.8 mm to (3.05, -4.50), turned to 90 degrees
- moved R11 9.08 mm to (1.80, -4.50), turned to 90 degrees
- moved D2 8.49 mm to (-1.27, -4.33)
- moved R10 7.41 mm to (0.55, -4.50), turned to 270 degrees
- moved R24 6.98 mm to (9.57, -3.80), turned to 180 degrees
- moved D1 6.79 mm to (12.0, 3.27), turned to 270 degrees
- moved C2 6.29 mm to (-8.18, 1.57), turned to 90 degrees
- moved C15 4.57 mm to (-2.27, -0.38), turned to 0 degrees
- moved R3 4.51 mm to (-3.75, -8.50), turned to 90 degrees
- moved LED0 3.54 mm to (-5.00, -8.50), turned to 90 degrees
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Connections:
- net CONSOLE_RX: no longer CON8.3
- net CONSOLE_TX: no longer CON8.2
- net GND: no longer CON8.6
- net TCK: no longer CON8.5
- net TMS: no longer CON8.4
- net TPWR: no longer CON8.1
Routing:
- net LED0: track 0.00 -> 13.2 mm
- net GND: track 0.00 -> 12.0 mm, vias 0 -> 10
- net LED2: track 0.00 -> 11.9 mm
- net LED1: track 0.00 -> 11.3 mm
- net VDD_3V3: track 0.00 -> 9.59 mm
- net N$9: track 0.00 -> 9.58 mm, vias 0 -> 2
- net SWITCH: track 0.00 -> 9.22 mm
- net N$8: track 0.00 -> 8.95 mm
- net N$3: track 0.00 -> 8.47 mm
- net VDD_5V: track 0.00 -> 6.30 mm
- net N$11: track 0.00 -> 5.10 mm
- net N$1: track 0.00 -> 5.00 mm
- net N$15: track 0.00 -> 4.90 mm
- net N$10: track 0.00 -> 4.87 mm
- net N$5: track 0.00 -> 1.60 mm
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- added copper zone on layer 16, net GND
Other:
- board size 45 x 20 mm -> 51 x 20 mm

Commit message: more routong
Parts:
- removed C16: 10nF, C_digikey:C0603
- moved R14 25.9 mm to (-23.2, -9.12), turned to 0 degrees
- moved Q2 24.0 mm to (-23.2, -7.17), turned to 90 degrees
- moved R21 12.8 mm to (-13.8, 0.80), turned to 180 degrees
- moved R13 11.9 mm to (-10.8, 1.15), turned to 180 degrees
- moved Q3 10.4 mm to (-10.4, 2.85), turned to 0 degrees
- moved R20 9.84 mm to (-13.8, 3.30)
- moved C14 8.28 mm to (-11.6, -1.00), turned to 270 degrees
- moved R22 7.11 mm to (-6.55, 7.85), turned to 270 degrees
- moved C11 5.59 mm to (-11.6, -8.50), turned to 270 degrees
- moved R24 4.65 mm to (13.7, -5.95), turned to 0 degrees
- moved C13 3.31 mm to (-11.6, -3.50), turned to 270 degrees
- moved C12 2.65 mm to (-11.6, -6.00)
- moved C8 2.50 mm to (-6.25, -3.50)
- moved C9 2.50 mm to (-6.25, -6.00)
- moved IC4 2.50 mm to (-9.00, -6.00)
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Connections:
- net GND: no longer C16.P$1
- net VDD_3V3: no longer C16.P$2
Routing:
- net VDD_5V: track 6.30 -> 46.2 mm, vias 0 -> 3
- net TPWR: track 0.00 -> 38.6 mm, vias 0 -> 2
- net PWR_BR: track 0.00 -> 36.5 mm, vias 0 -> 2
- net VDD_3V3: track 9.59 -> 34.8 mm
- net CONSOLE_RX: track 0.00 -> 20.4 mm
- net CONSOLE_TX: track 0.00 -> 17.8 mm, vias 0 -> 2
- net ITCK: track 0.00 -> 16.9 mm, vias 0 -> 2
- net IRST_SENSE: track 0.00 -> 16.8 mm, vias 0 -> 2
- net ITDI: track 0.00 -> 16.2 mm, vias 0 -> 2
- net IRST: track 0.00 -> 14.8 mm, vias 0 -> 2
- net TCK: track 0.00 -> 12.2 mm, vias 0 -> 2
- net TMS: track 0.00 -> 12.2 mm, vias 0 -> 2
- net GND: track 12.0 -> 0.49 mm, vias 10 -> 19
- net ITMS_DIR: track 0.00 -> 11.4 mm
- net XTPWR: track 0.00 -> 11.4 mm
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- added copper zone on layer 1, net GND

Commit message: more routing
Parts:
- added U$1: (no value), logo:DRAGON-30X13
Routing:
- net IRXD: track 0.00 -> 22.4 mm, vias 0 -> 2
- net ITXD: track 0.00 -> 21.7 mm, vias 0 -> 2
- net RST: track 0.00 -> 2.75 mm
- net GND: vias 19 -> 25
