File: 2.3/DCP23.sch (EAGLE design)
At the start: 0 parts

Commit message: blah
Parts:
- added C1, C2: 18pF, C_digikey:18PF-50V_5%_NP0-0603
- added CON1: USB-1, Connectors:USB-1
- added IC1: STM32F103CBT7, stm32:STM32F103CBT7
- added IC2: AP2127-3.3, linear regulators:AP2127-3.3
- added LED0, LED1, LED2, LED3: LED-0603, rc:LED-0603
- added Q1: 8 MHz, crystal:CRYSTAL-4P-8MHZ-3.2X5-4P
- added R1, R2, R3, R4: 1K, R_digikey:1K-5%-0603
Connections:
- new net GND: C1.2, C2.2, IC2.GND, LED0.C, LED1.C, LED2.C, LED3.C, Q1.GND
- new net LED0: IC1.PB2, R3.2
- new net LED1: IC1.PB10, R1.2
- new net LED2: IC1.PB11, R2.2
- new net N$1: C1.1, IC1.PD0, Q1.1
- new net N$2: LED0.A, R3.1
- new net N$3: C2.1, IC1.PD1, Q1.2
- new net N$4: LED2.A, R2.1
- new net N$5: LED1.A, R1.1
- new net N$6: LED3.A, R4.1
- new net SWITCH: IC1.PB12
- new net VBUS: IC1.PB13
- new net VDD_3V3: IC2.OUT, R4.2
- new net VDD_5V: IC2.EN, IC2.IN

Commit message: 2.3 schematic  completed
Parts:
- added C10, C11, C12, C13, C14, C17, C18, C19, C6, C7, C8, C9: 0.1µF, C_digikey:0.1µF-16V_10%_X7R-0603
- added C15: 1µF, C_digikey:1µF-10V_10%_X5R-0603
- added C16: 10nF, C_digikey:10NF-50V_10%_X7R-0603
- added C3, C4, C5: 4.7µF, C_digikey:4.7µF-6.3V_10%_X5R-0603
- added CON2: PINHEAD_1X02-2, pinhead:PINHEAD_1X02-2
- added CON3: CON-6P-SM06B, Connectors:CON-6P-SM06B
- added CON4: CON-2X5P, Connectors:CON-2X5P
- added CON5: CON-6P-DF13, Connectors:CON-6P-DF13
- added CON6: PINHEAD_1X04-2.54, pinhead:PINHEAD_1X04-2.54
- added CON7: PINHEAD_1X03-2.54, pinhead:PINHEAD_1X03-2.54
- added CON8: PINHEAD_1X06-2.54, pinhead:PINHEAD_1X06-2.54
- added D1: PRTR5V0U2X, TVS_diodes:PRTR5V0U2X
- added IC3, IC4, IC5, IC6: 74LVC2T45, misc:74LVC2T45
- added Q2: DMG1023UV-7, mosfet:DMG1023UV-7
- added Q3: DMG1024UV-7, mosfet:DMG1024UV-7
- added R10: 4K7, R_digikey:4K7-1%-0603
- added R11, R12, R13, R14, R24: 10K, R_digikey:10K-5%-0603
- added R15, R16, R17, R18, R19, R20, R21, R23: 120R, R_digikey:120R-1%-0603
- added R22: 0, R_digikey:0R-5%-0603
- added R5, R6: 22R, rc:R-5%-0603
- added R7: 1K5, rc:R-5%-0603
- added SW1: TACT_SWITCH-FSMSM, misc:TACT_SWITCH-FSMSM
Connections:
- removed net VBUS: IC1.PB13
- new net !RST: IC1.NRST
- new net CONSOLE_RX: CON3.3, CON5.5, CON8.3, R23.2
- new net CONSOLE_TX: CON3.2, CON5.4, CON8.2, R20.2
- new net IRST: IC1.PA2, Q3Q2.G
- new net IRST_SENSE: IC1.PA7, Q3Q1.D
- new net IRXD: IC1.PA10, IC5.2A
- new net ITCK: IC1.PA5, IC4.1A
- new net ITDI: IC1.PA3, IC4.2A
- new net ITDO: IC1.PA6, IC5.1A
- new net ITMS: IC1.PA4, IC6.2A
- new net ITMS_DIR: IC1.PA1, IC6.DIR
- new net ITXD: IC1.PA9, IC3.2A
- new net N$10: CON1.D-, CON6.2, R6.2
- new net N$11: CON1.D+, CON6.1, R5.2
- new net N$12: Q2Q1.S, Q2Q2.S, R14.1
- new net N$13: CON5.1, R22.2
- new net N$15: CON2.1, IC1.BOOT0, R12.1
- new net N$7: IC1.PA8, R7.1
- new net N$8: D1.D2, IC1.PA11, R6.1
- new net N$9: D1.D1, IC1.PA12, R5.1, R7.2
- new net PWR_BR: IC1.PB1, Q2Q1.G, Q2Q2.G, R14.2
- new net RST: CON4.10, R15.2
- new net SWCLK: CON7.3, IC1.PA14
- new net SWDIO: CON7.1, IC1.PA13
- new net TCK: CON3.5, CON4.4, CON8.5, R18.2
- new net TDI: CON4.8, R16.2
- new net TDO: CON4.6, R17.2
- new net TMS: CON3.4, CON4.2, CON8.4, R19.2
- new net TPWR: CON3.1, CON4.1, CON8.1, Q2Q2.D, R10.2, R21.2
- new net TRACESWO: IC1.PB3
- new net VBUS1: C6.2, IC1.PB0, R10.1, R11.2
- new net XRST: Q3Q1.G, Q3Q2.D, R13.1, R15.1
- new net XRXD: IC5.2B, R20.1
- new net XTCK: IC4.1B, R18.1
- new net XTDI: IC4.2B, R16.1
- new net XTDO: IC5.1B, R17.1
- new net XTMS: IC6.2B, R19.1
- new net XTPWR: C11.2, C12.2, C13.2, C14.2, IC3.VCCB, IC4.VCCB, IC5.VCCB, IC6.VCCB, R13.2, R21.1
- new net XTXD: IC3.2B, R23.1
- net GND: now also C10.2, C11.1, C12.1, C13.1, C14.1, C15.1, C16.1, C17.2, C18.1, C19.2, C3.1, C4.1, C5.2, C6.1, C7.2, C8.2, C9.2, CON1.GND, CON3.6, CON3.G1, CON3.G2, CON4.3, CON4.5, CON4.9, CON5.G1, CON5.G2, CON6.4, CON7.2, CON8.6, D1.C, IC1.VSS@1, IC1.VSS@2, IC1.VSSA, IC3.1A, IC3.1B, IC3.GND, IC4.GND, IC5.DIR, IC5.GND, IC6.1A, IC6.1B, IC6.GND, Q3Q1.S, Q3Q2.S, R11.1, R12.2, SW1.2
- net SWITCH: now also R24.1, SW1.1
- net VDD_3V3: now also C10.1, C15.2, C16.2, C17.1, C18.2, C19.1, C4.2, C5.1, C7.1, C8.1, C9.1, CON2.2, IC1.PB4, IC1.PB5, IC1.PB6, IC1.VBAT, IC1.VDD@1, IC1.VDD@2, IC1.VDD@3, IC1.VDDA, IC3.DIR, IC3.VCCA, IC4.DIR, IC4.VCCA, IC5.VCCA, IC6.VCCA, Q2Q1.D, R24.2
- net VDD_5V: now also C3.2, CON1.VBUS, CON6.3, D1.A, IC1.PB13, R22.1
Other:
- note added: "->"
- note added: "<-"
- note added: "<- DIR = GND -> DIR = VCC"
- note added: "<->"
- note added: "CON7 is for firmware flashing"
- note added: "HIGH on DIR allows transmission from nA to nB LOW on DIR allows transmission from nB to nA"
- note added: "PB13 is FT pin No divider needed"
- note added: "R8, R9 should not be populated"
- note added: "SWCLK"
- note added: "SWDIO"
- note added: "TMS = SWDIO TDO = TRACESWO TCK = SWCLK"
- moved on the sheet: C1, C2, CON1, IC1, IC2, LED0, LED1, LED2, LED3, Q1, R1, R2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

Commit message: Some routing
Parts:
- added D2: BAT30SWFILM, Diodes:BAT30SWFILM
Connections:
- net GND: now also CON6.1, D2.A; no longer CON6.4
- net N$10: now also CON6.3; no longer CON6.2
- net N$11: now also CON6.2; no longer CON6.1
- net VBUS1: now also D2.COMMON
- net VDD_3V3: now also D2.C
- net VDD_5V: now also CON6.4; no longer CON6.3
Changed lines of the file:
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@@
 <part name="GND35" library="supply_symbols" library_urn="urn:adsk.eagle:library:5017758" deviceset="GND" device="" value="GND"/>
 <part name="+P17" library="supply_symbols" library_urn="urn:adsk.eagle:library:5017758" deviceset="3.3V" device=""/>
+<part name="GND11" library="supply_symbols" library_urn="urn:adsk.eagle:library:5017758" deviceset="GND" device="" value="GND"/>
+<part name="+P18" library="supply_symbols" library_urn="urn:adsk.eagle:library:5017758" deviceset="5V" device=""/>
+<part name="D2" library="Diodes" library_urn="urn:adsk.eagle:library:2473263" deviceset="BAT30SWFILM" device="" package3d_urn="urn:adsk.eagle:package:7365870/2"/>
+<part name="+P19" library="supply_symbols" library_urn="urn:adsk.eagle:library:5017758" deviceset="3.3V" device=""/>
+<part name="GND36" library="supply_symbols" library_urn="urn:adsk.eagle:library:5017758" deviceset="GND" device="" value="GND"/>
 </parts>
 <sheets>
@@
 <attribute name="VALUE" x="139.7" y="173.736" size="1.27" layer="96" font="vector" ratio="15" align="center"/>
 </instance>
+<instance part="GND11" gate="1" x="147.32" y="124.46" smashed="yes">
+<attribute name="VALUE" x="147.32" y="123.19" size="1.27" layer="96" font="vector" ratio="15" align="center"/>
+</instance>
+<instance part="+P18" gate="G$1" x="142.24" y="139.7" smashed="yes">
+<attribute name="VALUE" x="142.24" y="143.256" size="1.27" layer="96" font="vector" ratio="15" align="center"/>
+</instance>
+<instance part="D2" gate="G$1" x="40.64" y="50.8" smashed="yes">
+<attribute name="NAME" x="37.592" y="50.8" size="1.27" layer="95" font="vector" ratio="15" rot="R90" align="center"/>
+<attribute name="MANF#" x="38.862" y="50.8" size="0.762" layer="95" font="vector" ratio="15" rot="R270" align="center"/>
+</instance>
+<instance part="+P19" gate="G$1" x="40.64" y="58.42" smashed="yes">
+<attribute name="VALUE" x="40.64" y="61.976" size="1.27" layer="96" font="vector" ratio="15" align="center"/>
+</instance>
+<instance part="GND36" gate="1" x="40.64" y="33.02" smashed="yes">
+<attribute name="VALUE" x="40.64" y="31.75" size="1.27" layer="96" font="vector" ratio="15" align="center"/>
+</instance>
 </instances>
 <busses>
@@
 <segment>
 <pinref part="CON1" gate="G$1" pin="GND"/>
-<wire x1="137.16" y1="129.54" x2="137.16" y2="111.76" width="0.1524" layer="91"/>
-<wire x1="137.16" y1="111.76" x2="147.32" y2="111.76" width="0.1524" layer="91"/>
 <pinref part="GND9" gate="1" pin="GND"/>
 <wire x1="137.16" y1="111.76" x2="137.16" y2="109.22" width="0.1524" layer="91"/>
-<junction x="137.16" y="111.76"/>
-<wire x1="137.16" y1="129.54" x2="137.16" y2="137.16" width="0.1524" layer="91"/>
-<pinref part="CON6" gate="G$1" pin="4"/>
-<wire x1="137.16" y1="137.16" x2="149.86" y2="137.16" width="0.1524" layer="91"/>
+<wire x1="137.16" y1="111.76" x2="147.32" y2="111.76" width="0.1524" layer="91"/>
 </segment>
 <segment>
@@
 <pinref part="SW1" gate="G$1" pin="2"/>
 <wire x1="154.94" y1="154.94" x2="152.4" y2="154.94" width="0.1524" layer="91"/>
+</segment>
+<segment>
+<pinref part="GND11" gate="1" pin="GND"/>
+<wire x1="147.32" y1="127" x2="147.32" y2="129.54" width="0.1524" layer="91"/>
+<pinref part="CON6" gate="G$1" pin="1"/>
+<wire x1="147.32" y1="129.54" x2="149.86" y2="129.54" width="0.1524" layer="91"/>
+</segment>
+<segment>
+<pinref part="GND36" gate="1" pin="GND"/>
+<pinref part="D2" gate="G$1" pin="A"/>
+<wire x1="40.64" y1="35.56" x2="40.64" y2="45.72" width="0.1524" layer="91"/>
 </segment>
 </net>
@@
 <wire x1="124.46" y1="114.3" x2="104.14" y2="114.3" width="0.1524" layer="91"/>
 <wire x1="104.14" y1="114.3" x2="104.14" y2="106.68" width="0.1524" layer="91"/>
-<wire x1="139.7" y1="132.08" x2="139.7" y2="114.3" width="0.1524" layer="91"/>
-<junction x="139.7" y="114.3"/>
-<pinref part="CON6" gate="G$1" pin="3"/>
-<wire x1="149.86" y1="134.62" x2="139.7" y2="134.62" width="0.1524" layer="91"/>
-<wire x1="139.7" y1="134.62" x2="139.7" y2="132.08" width="0.1524" layer="91"/>
 <pinref part="IC1" gate="G$1" pin="PB13"/>
 <wire x1="86.36" y1="101.6" x2="88.9" y2="101.6" width="0.1524" layer="91"/>
@@
 <pinref part="+P16" gate="G$1" pin="VDD_5V"/>
 <wire x1="142.24" y1="99.06" x2="142.24" y2="101.6" width="0.1524" layer="91"/>
+</segment>
+<segment>
+<pinref part="CON6" gate="G$1" pin="4"/>
+<wire x1="149.86" y1="137.16" x2="142.24" y2="137.16" width="0.1524" layer="91"/>
+<pinref part="+P18" gate="G$1" pin="VDD_5V"/>
+<wire x1="142.24" y1="137.16" x2="142.24" y2="139.7" width="0.1524" layer="91"/>
 </segment>
 </net>
@@
 <wire x1="139.7" y1="167.64" x2="139.7" y2="170.18" width="0.1524" layer="91"/>
 </segment>
+<segment>
+<pinref part="+P19" gate="G$1" pin="VDD_3V3"/>
+<pinref part="D2" gate="G$1" pin="C"/>
+<wire x1="40.64" y1="58.42" x2="40.64" y2="55.88" width="0.1524" layer="91"/>
+</segment>
 </net>
 <net name="N$5" class="0">
@@
 <wire x1="142.24" y1="116.84" x2="137.16" y2="116.84" width="0.1524" layer="91"/>
 <junction x="142.24" y="116.84"/>
-<pinref part="CON6" gate="G$1" pin="2"/>
 <wire x1="142.24" y1="132.08" x2="142.24" y2="116.84" width="0.1524" layer="91"/>
-<wire x1="149.86" y1="132.08" x2="142.24" y2="132.08" width="0.1524" layer="91"/>
+<wire x1="142.24" y1="132.08" x2="142.24" y2="134.62" width="0.1524" layer="91"/>
+<pinref part="CON6" gate="G$1" pin="3"/>
+<wire x1="142.24" y1="134.62" x2="149.86" y2="134.62" width="0.1524" layer="91"/>
 </segment>
 </net>
@@
 <wire x1="144.78" y1="129.54" x2="144.78" y2="119.38" width="0.1524" layer="91"/>
 <junction x="144.78" y="119.38"/>
-<pinref part="CON6" gate="G$1" pin="1"/>
-<wire x1="144.78" y1="129.54" x2="149.86" y2="129.54" width="0.1524" layer="91"/>
+<wire x1="144.78" y1="129.54" x2="144.78" y2="132.08" width="0.1524" layer="91"/>
+<wire x1="144.78" y1="132.08" x2="147.32" y2="132.08" width="0.1524" layer="91"/>
+<pinref part="CON6" gate="G$1" pin="2"/>
+<wire x1="147.32" y1="132.08" x2="149.86" y2="132.08" width="0.1524" layer="91"/>
 </segment>
 </net>
@@
 <pinref part="IC1" gate="G$1" pin="PB0"/>
 <wire x1="58.42" y1="68.58" x2="58.42" y2="86.36" width="0.1524" layer="91"/>
-</segment>
-</net>
+<pinref part="D2" gate="G$1" pin="COMMON"/>
+<wire x1="45.72" y1="50.8" x2="43.18" y2="50.8" width="0.1524" layer="91"/>
+</segment>
+</net>

Commit message: more routing
Parts:
- removed CON8: PINHEAD_1X06-2.54, pinhead:PINHEAD_1X06-2.54
- added CON10: PINHEAD_2X03-PTH-2.54, pinhead:PINHEAD_2X03-PTH-2.54
Connections:
- net CONSOLE_RX: no longer CON8.3
- net CONSOLE_TX: no longer CON8.2
- net GND: no longer CON8.6
- net TCK: no longer CON8.5
- net TMS: no longer CON8.4
- net TPWR: no longer CON8.1
Changed lines of the file:
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@@
 <part name="CON7" library="pinhead" library_urn="urn:adsk.eagle:library:2540341" deviceset="PINHEAD_1X03" device="-2.54" package3d_urn="urn:adsk.eagle:package:2540386/2"/>
 <part name="GND34" library="supply_symbols" library_urn="urn:adsk.eagle:library:5017758" deviceset="GND" device="" value="GND"/>
-<part name="CON8" library="pinhead" library_urn="urn:adsk.eagle:library:2540341" deviceset="PINHEAD_1X06" device="-2.54" package3d_urn="urn:adsk.eagle:package:2540381/1"/>
 <part name="SW1" library="misc" library_urn="urn:adsk.eagle:library:5347860" deviceset="TACT_SWITCH" device="-FSMSM" package3d_urn="urn:adsk.eagle:package:8723450/2"/>
 <part name="R24" library="R_digikey" library_urn="urn:adsk.eagle:library:2539499" deviceset="10K" device="-0603" package3d_urn="urn:adsk.eagle:package:2539515/2" technology="-5%" value="10K"/>
@@
 <part name="+P19" library="supply_symbols" library_urn="urn:adsk.eagle:library:5017758" deviceset="3.3V" device=""/>
 <part name="GND36" library="supply_symbols" library_urn="urn:adsk.eagle:library:5017758" deviceset="GND" device="" value="GND"/>
+<part name="CON10" library="pinhead" library_urn="urn:adsk.eagle:library:2540341" deviceset="PINHEAD_2X03" device="-PTH-2.54" package3d_urn="urn:adsk.eagle:package:8729607/1"/>
 </parts>
 <sheets>
@@
 <attribute name="VALUE" x="104.14" y="133.35" size="1.27" layer="96" font="vector" ratio="15" align="center"/>
 </instance>
-<instance part="CON8" gate="G$1" x="160.02" y="20.32" smashed="yes" rot="MR0">
-<attribute name="NAME" x="157.48" y="39.37" size="1.778" layer="95" font="vector" ratio="15" rot="MR0" align="center"/>
-</instance>
 <instance part="SW1" gate="G$1" x="147.32" y="154.94" smashed="yes">
 <attribute name="NAME" x="147.32" y="157.48" size="1.778" layer="95" font="vector" ratio="10" align="center"/>
@@
 <instance part="GND36" gate="1" x="40.64" y="33.02" smashed="yes">
 <attribute name="VALUE" x="40.64" y="31.75" size="1.27" layer="96" font="vector" ratio="15" align="center"/>
+</instance>
+<instance part="CON10" gate="G$1" x="177.8" y="25.4" smashed="yes">
+<attribute name="NAME" x="184.404" y="36.83" size="1.778" layer="95" font="vector" ratio="15" align="center"/>
 </instance>
 </instances>
@@
 <wire x1="147.32" y1="35.56" x2="147.32" y2="43.18" width="0.1524" layer="91"/>
 <junction x="147.32" y="43.18"/>
-<pinref part="CON8" gate="G$1" pin="6"/>
 <wire x1="149.86" y1="35.56" x2="152.4" y2="35.56" width="0.1524" layer="91"/>
 </segment>
@@
 <wire x1="149.86" y1="22.86" x2="147.32" y2="22.86" width="0.1524" layer="91"/>
 <label x="147.32" y="22.86" size="1.27" layer="95" rot="R180" xref="yes"/>
-<pinref part="CON8" gate="G$1" pin="1"/>
 <wire x1="149.86" y1="22.86" x2="152.4" y2="22.86" width="0.1524" layer="91"/>
 </segment>
@@
 <wire x1="137.16" y1="60.96" x2="137.16" y2="25.4" width="0.1524" layer="91"/>
 <wire x1="137.16" y1="25.4" x2="149.86" y2="25.4" width="0.1524" layer="91"/>
-<pinref part="CON8" gate="G$1" pin="2"/>
 <wire x1="149.86" y1="25.4" x2="152.4" y2="25.4" width="0.1524" layer="91"/>
 </segment>
@@
 <wire x1="139.7" y1="58.42" x2="139.7" y2="27.94" width="0.1524" layer="91"/>
 <wire x1="139.7" y1="27.94" x2="149.86" y2="27.94" width="0.1524" layer="91"/>
-<pinref part="CON8" gate="G$1" pin="3"/>
 <wire x1="149.86" y1="27.94" x2="152.4" y2="27.94" width="0.1524" layer="91"/>
 </segment>
@@
 <wire x1="157.48" y1="53.34" x2="144.78" y2="53.34" width="0.1524" layer="91"/>
 <label x="116.84" y="53.34" size="1.27" layer="95" rot="R180" xref="yes"/>
-<pinref part="CON8" gate="G$1" pin="5"/>
 <wire x1="144.78" y1="53.34" x2="116.84" y2="53.34" width="0.1524" layer="91"/>
 <wire x1="152.4" y1="33.02" x2="144.78" y2="33.02" width="0.1524" layer="91"/>
@@
 <wire x1="157.48" y1="55.88" x2="142.24" y2="55.88" width="0.1524" layer="91"/>
 <label x="116.84" y="55.88" size="1.27" layer="95" rot="R180" xref="yes"/>
-<pinref part="CON8" gate="G$1" pin="4"/>
 <wire x1="142.24" y1="55.88" x2="116.84" y2="55.88" width="0.1524" layer="91"/>
 <wire x1="152.4" y1="30.48" x2="142.24" y2="30.48" width="0.1524" layer="91"/>
@@
 </nets>
 </sheet>
+<sheet>
+<plain>
+</plain>
+<instances>
+</instances>
+<busses>
+</busses>
+<nets>
+</nets>
+</sheet>

Commit message: more routong
Parts:
- removed C16: 10nF, C_digikey:10NF-50V_10%_X7R-0603
Connections:
- net GND: no longer C16.1
- net VDD_3V3: no longer C16.2
Changed lines of the file:
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@@
 <part name="FRAME1" library="frames" library_urn="urn:adsk.eagle:library:229" deviceset="A4L-LOC" device=""/>
 <part name="IC1" library="stm32" library_urn="urn:adsk.eagle:library:2473361" deviceset="STM32F103CBT7" device="" package3d_urn="urn:adsk.eagle:package:2473350/3"/>
-<part name="CON1" library="Connectors" library_urn="urn:adsk.eagle:library:3750510" deviceset="USB" device="-1" package3d_urn="urn:adsk.eagle:package:1041165/1"/>
+<part name="CON1" library="Connectors" library_urn="urn:adsk.eagle:library:3750510" deviceset="USB" device="-1" package3d_urn="urn:adsk.eagle:package:1041165/2"/>
 <part name="Q1" library="crystal" library_urn="urn:adsk.eagle:library:2539107" deviceset="CRYSTAL-4P" device="-3.2X5-4P" package3d_urn="urn:adsk.eagle:package:2539116/3" technology="-8MHZ" value="8 MHz"/>
 <part name="C1" library="C_digikey" library_urn="urn:adsk.eagle:library:2539367" deviceset="18PF" device="-0603" package3d_urn="urn:adsk.eagle:package:2539381/2" technology="-50V_5%_NP0" value="18pF"/>
@@
 <part name="+P7" library="supply_symbols" library_urn="urn:adsk.eagle:library:5017758" deviceset="3.3V" device=""/>
 <part name="C15" library="C_digikey" library_urn="urn:adsk.eagle:library:2539367" deviceset="1µF" device="-0603" package3d_urn="urn:adsk.eagle:package:2539381/2" technology="-10V_10%_X5R" value="1µF"/>
-<part name="C16" library="C_digikey" library_urn="urn:adsk.eagle:library:2539367" deviceset="10NF" device="-0603" package3d_urn="urn:adsk.eagle:package:2539381/2" technology="-50V_10%_X7R" value="10nF"/>
 <part name="GND23" library="supply_symbols" library_urn="urn:adsk.eagle:library:5017758" deviceset="GND" device="" value="GND"/>
-<part name="GND24" library="supply_symbols" library_urn="urn:adsk.eagle:library:5017758" deviceset="GND" device="" value="GND"/>
 <part name="GND25" library="supply_symbols" library_urn="urn:adsk.eagle:library:5017758" deviceset="GND" device="" value="GND"/>
 <part name="+P8" library="supply_symbols" library_urn="urn:adsk.eagle:library:5017758" deviceset="3.3V" device=""/>
@@
 <part name="R20" library="R_digikey" library_urn="urn:adsk.eagle:library:2539499" deviceset="120R" device="-0603" package3d_urn="urn:adsk.eagle:package:2539515/2" technology="-1%" value="120R"/>
 <part name="CON4" library="Connectors" library_urn="urn:adsk.eagle:library:3750510" deviceset="CON-2X5P" device="" package3d_urn="urn:adsk.eagle:package:8721870/2"/>
-<part name="CON5" library="Connectors" library_urn="urn:adsk.eagle:library:3750510" deviceset="CON-6P" device="-DF13" package3d_urn="urn:adsk.eagle:package:8719648/2"/>
+<part name="CON5" library="Connectors" library_urn="urn:adsk.eagle:library:3750510" deviceset="CON-6P" device="-DF13" package3d_urn="urn:adsk.eagle:package:8719648/3"/>
 <part name="+P15" library="supply_symbols" library_urn="urn:adsk.eagle:library:5017758" deviceset="3.3V" device=""/>
 <part name="GND32" library="supply_symbols" library_urn="urn:adsk.eagle:library:5017758" deviceset="GND" device="" value="GND"/>
@@
 <part name="+P19" library="supply_symbols" library_urn="urn:adsk.eagle:library:5017758" deviceset="3.3V" device=""/>
 <part name="GND36" library="supply_symbols" library_urn="urn:adsk.eagle:library:5017758" deviceset="GND" device="" value="GND"/>
-<part name="CON10" library="pinhead" library_urn="urn:adsk.eagle:library:2540341" deviceset="PINHEAD_2X03" device="-PTH-2.54" package3d_urn="urn:adsk.eagle:package:8729607/1"/>
+<part name="CON10" library="pinhead" library_urn="urn:adsk.eagle:library:2540341" deviceset="PINHEAD_2X03" device="-PTH-2.54" package3d_urn="urn:adsk.eagle:package:8729607/3"/>
 </parts>
 <sheets>
@@
 <attribute name="VOLTAGE" x="9.906" y="103.886" size="0.762" layer="96" rot="R90" align="bottom-center"/>
 </instance>
-<instance part="C16" gate="G$1" x="15.24" y="101.6" smashed="yes" rot="R90">
-<attribute name="NAME" x="16.129" y="102.87" size="1.27" layer="95" rot="R90" align="center-left"/>
-<attribute name="VALUE" x="14.986" y="100.33" size="0.762" layer="96" rot="R90" align="bottom-right"/>
-<attribute name="PACKAGE" x="15.748" y="99.568" size="0.508" layer="97" rot="R270" align="center"/>
-<attribute name="VOLTAGE" x="14.986" y="103.886" size="0.762" layer="96" rot="R90" align="bottom-center"/>
-</instance>
 <instance part="GND23" gate="1" x="10.16" y="93.98" smashed="yes">
 <attribute name="VALUE" x="10.16" y="92.71" size="1.27" layer="96" font="vector" ratio="15" align="center"/>
-</instance>
-<instance part="GND24" gate="1" x="15.24" y="93.98" smashed="yes">
-<attribute name="VALUE" x="15.24" y="92.71" size="1.27" layer="96" font="vector" ratio="15" align="center"/>
 </instance>
 <instance part="GND25" gate="1" x="20.32" y="109.22" smashed="yes" rot="R270">
@@
 <pinref part="GND23" gate="1" pin="GND"/>
 <wire x1="10.16" y1="96.52" x2="10.16" y2="99.06" width="0.1524" layer="91"/>
-</segment>
-<segment>
-<pinref part="C16" gate="G$1" pin="1"/>
-<pinref part="GND24" gate="1" pin="GND"/>
-<wire x1="15.24" y1="96.52" x2="15.24" y2="99.06" width="0.1524" layer="91"/>
 </segment>
 <segment>
@@
 <wire x1="15.24" y1="106.68" x2="10.16" y2="106.68" width="0.1524" layer="91"/>
 <wire x1="10.16" y1="104.14" x2="10.16" y2="106.68" width="0.1524" layer="91"/>
-<pinref part="C16" gate="G$1" pin="2"/>
-<wire x1="15.24" y1="104.14" x2="15.24" y2="106.68" width="0.1524" layer="91"/>
-<junction x="15.24" y="106.68"/>
 <pinref part="+P8" gate="G$1" pin="VDD_3V3"/>
 <wire x1="10.16" y1="109.22" x2="10.16" y2="106.68" width="0.1524" layer="91"/>

Commit message: more routing
Other:
- moved on the sheet: CON10
Changed lines of the file:
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@@
 <attribute name="VALUE" x="40.64" y="31.75" size="1.27" layer="96" font="vector" ratio="15" align="center"/>
 </instance>
-<instance part="CON10" gate="G$1" x="177.8" y="25.4" smashed="yes">
-<attribute name="NAME" x="184.404" y="36.83" size="1.778" layer="95" font="vector" ratio="15" align="center"/>
+<instance part="CON10" gate="G$1" x="170.18" y="25.4" smashed="yes">
+<attribute name="NAME" x="176.784" y="36.83" size="1.778" layer="95" font="vector" ratio="15" align="center"/>
 </instance>
 </instances>
